File: KiCad-PCB/keyboard.kicad_pcb (KiCad board)
At the start: 2 copper layers, 408 x 110.3 mm, 307 parts, among them J1 Conn_01x04_Female, SW1 SW_Push, U1 ATmega32U4-AU, Y1 Crystal_GND24_Small

Commit message: Case lasercut update
Parts:
- added G***: LOGO, dd:jf, B.Cu at (92.1, -11.1)
Routing:
- net +5V: track 743.0 -> 749.4 mm, vias 3 -> 2
- net D+: track 72.2 -> 73.4 mm
- net D-: track 65.9 -> 66.9 mm
Other:
- board size 408 x 110.3 mm -> 408 x 111.9 mm
